File: hardware/ym2612_player/audio.kicad_sch (KiCad schematic)
At the start: 55 parts, among them J2 1/4" TRS balanced out L, J3 1/4" TRS balanced out R, J4 3.5 mm headphones (front), U6 OPA2350UA, U7 OPA2350UA, U8 NJM4556AD

Commit message: Rev A PCB layout and PCBWay files
Board is 240 x 120 mm, 2 layers, placed by tools/layout.py and routed with
Freerouting (tools/route.py). DRC in KiCad 10: 0 errors, 0 unconnected,
matches the schematic. Adds Gerbers, BOM and placement (CPL) files for a
PCBWay turnkey order, and a top-view picture.

Also: volume slider moves off the board onto a 6-pin JST XH plug (J4), and
the Pico Plus 2 footprint now has its pads and outline in the right place.

Co-Authored-By: Claude Opus 5.5 (1M context) <noreply@anthropic.com>
Claude-Session: https://claude.ai/code/session_01JeM5NcWqyQVA3DixJkw6Wg
Parts:
- removed C34: 100nF, Capacitor_SMD:C_0603_1608Metric, symbol Device:C
- C20: renamed from RV1; value 10k audio, dual slide -> 1uF; footprint (none) -> Capacitor_SMD:C_1206_3216Metric; symbol Device:R_Potentiometer_Dual_Separate -> Device:C; MPN PTA2044-2015DPA103 -> (none); Spec Bourns 20 mm travel dual-gang slide pot, 10k audio taper, 1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 -> film or X7R 1206, 25V
- C21: renamed from U8; value NJM4556AD -> 220uF; footprint Package_DIP:DIP-8_W7.62mm -> Capacitor_SMD:CP_Elec_6.3x7.7; symbol Amplifier_Operational:NJM4556A -> Device:C_Polarized; MPN NJM4556AD -> (none); Spec dual high-current op-amp, DIP-8 -> electrolytic, 10V
- C22: renamed from R34; value 2.2k -> 1uF; footprint Resistor_SMD:R_0603_1608Metric -> Capacitor_SMD:C_1206_3216Metric; symbol Device:R -> Device:C; Spec 1%, 0603 -> film or C0G/X7R 1206, 25V (film preferred)
- C23: renamed from R36; value 100k -> 470pF; footprint Resistor_SMD:R_0603_1608Metric -> Capacitor_SMD:C_0603_1608Metric; symbol Device:R -> Device:C; Spec 1%, 0603 -> C0G, 50V
- C24: renamed from R39; value 100 -> 10uF; footprint Resistor_SMD:R_0603_1608Metric -> Capacitor_SMD:CP_Elec_5x5.4; symbol Device:R -> Device:C_Polarized; Spec 1%, 0603 -> electrolytic, 16V, low-leakage
- C25: renamed from R41; value 100 -> 10uF; footprint Resistor_SMD:R_0603_1608Metric -> Capacitor_SMD:CP_Elec_5x5.4; symbol Device:R -> Device:C_Polarized; Spec 1%, 0603 -> electrolytic, 16V, low-leakage
- C26: renamed from R43; value 0 -> 10uF; footprint Resistor_SMD:R_0603_1608Metric -> Capacitor_SMD:CP_Elec_5x5.4; symbol Device:R -> Device:C_Polarized; Spec 0 ohm, 0603 (ground lift option) -> electrolytic, 16V
- C27: renamed from C26; value 10uF -> 1uF; footprint Capacitor_SMD:CP_Elec_5x5.4 -> Capacitor_SMD:C_1206_3216Metric; symbol Device:C_Polarized -> Device:C; Spec electrolytic, 16V -> film or X7R 1206, 25V
- C28: renamed from R44; value 100k -> 220uF; footprint Resistor_SMD:R_0603_1608Metric -> Capacitor_SMD:CP_Elec_6.3x7.7; symbol Device:R -> Device:C_Polarized; Spec 1%, 0603 -> electrolytic, 10V
- C29: renamed from U8; value NJM4556AD -> 100nF; footprint Package_DIP:DIP-8_W7.62mm -> Capacitor_SMD:C_0603_1608Metric; symbol Amplifier_Operational:NJM4556A -> Device:C; MPN NJM4556AD -> (none); Spec dual high-current op-amp, DIP-8 -> X7R, 16V
- C32: renamed from C31; value 100nF -> 10uF; footprint Capacitor_SMD:C_0603_1608Metric -> Capacitor_SMD:C_0805_2012Metric; Spec X7R, 16V -> X5R, 10V, 0805
- C33: renamed from R48; value 10k -> 47uF; footprint Resistor_SMD:R_0603_1608Metric -> Capacitor_SMD:CP_Elec_5x5.4; symbol Device:R -> Device:C_Polarized; Spec 1%, 0603 -> electrolytic, 16V
- C34: renamed from C33; value 47uF -> 100nF; footprint Capacitor_SMD:CP_Elec_5x5.4 -> Capacitor_SMD:C_0603_1608Metric; symbol Device:C_Polarized -> Device:C; Spec electrolytic, 16V -> X7R, 16V
- J3: renamed from R42; value 100k -> 1/4" TRS balanced out R; footprint Resistor_SMD:R_0603_1608Metric -> Connector_Audio:Jack_6.35mm_Neutrik_NMJ6HCD2_Horizontal; symbol Device:R -> Connector_Audio:AudioJack3_SwitchTR; MPN (none) -> NMJ6HCD2; Spec 1%, 0603 -> Neutrik 1/4in stereo jack, horizontal PCB. The footprint's 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
- J4: renamed from R45; value 10 -> Volume slider (dual 10k audio taper, in the case); footprint Resistor_SMD:R_0603_1608Metric -> Connector_JST:JST_XH_B6B-XH-A_1x06_P2.50mm_Vertical; symbol Device:R -> Connector_Generic:Conn_01x06; MPN (none) -> B6B-XH-A(LF)(SN); Spec 1%, 0603 -> JST XH 6-pin header. Wire a dual 10k audio-taper slide pot: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
- J5: renamed from R46; value 10k -> 3.5 mm headphones (front); footprint Resistor_SMD:R_0603_1608Metric -> Connector_Audio:Jack_3.5mm_CUI_SJ1-3523N_Horizontal; symbol Device:R -> Connector_Audio:AudioJack3; MPN (none) -> SJ1-3523N; Spec 1%, 0603 -> CUI 3.5 mm stereo jack, horizontal
- R31: renamed from C20; value 1uF -> 100k; footprint Capacitor_SMD:C_1206_3216Metric -> Resistor_SMD:R_0603_1608Metric; symbol Device:C -> Device:R; Spec film or X7R 1206, 25V -> 1%, 0603
- R32: renamed from C21; value 220uF -> 10; footprint Capacitor_SMD:CP_Elec_6.3x7.7 -> Resistor_SMD:R_0603_1608Metric; symbol Device:C_Polarized -> Device:R; Spec electrolytic, 10V -> 1%, 0603
- R33: renamed from R32; value 10 -> 10k
- R34: renamed from R33; value 10k -> 2.2k
- R35: renamed from C22; value 1uF -> 47k; footprint Capacitor_SMD:C_1206_3216Metric -> Resistor_SMD:R_0603_1608Metric; symbol Device:C -> Device:R; Spec film or C0G/X7R 1206, 25V (film preferred) -> 1%, 0603
- R36: renamed from R35; value 47k -> 100k
- R37: renamed from U6; value OPA2350UA -> 10k; footprint Package_SO:SOIC-8_3.9x4.9mm_P1.27mm -> Resistor_SMD:R_0603_1608Metric; symbol Amplifier_Operational:OPA2340 -> Device:R; MPN OPA2350UA -> (none); Spec dual rail-to-rail op-amp, 2.7-5.5V -> 1%, 0603
- R39: renamed from U7; value OPA2350UA -> 100; footprint Package_SO:SOIC-8_3.9x4.9mm_P1.27mm -> Resistor_SMD:R_0603_1608Metric; symbol Amplifier_Operational:OPA2340 -> Device:R; MPN OPA2350UA -> (none); Spec dual rail-to-rail op-amp, 2.7-5.5V -> 1%, 0603
- R40: renamed from C24; value 10uF -> 100k; footprint Capacitor_SMD:CP_Elec_5x5.4 -> Resistor_SMD:R_0603_1608Metric; symbol Device:C_Polarized -> Device:R; Spec electrolytic, 16V, low-leakage -> 1%, 0603
- R41: renamed from R40; value 100k -> 100
- R42: renamed from C25; value 10uF -> 100k; footprint Capacitor_SMD:CP_Elec_5x5.4 -> Resistor_SMD:R_0603_1608Metric; symbol Device:C_Polarized -> Device:R; Spec electrolytic, 16V, low-leakage -> 1%, 0603
- R43: renamed from J3; value 1/4" TRS balanced out R -> 0; footprint Connector_Audio:Jack_6.35mm_Neutrik_NMJ6HCD2_Horizontal -> Resistor_SMD:R_0603_1608Metric; symbol Connector_Audio:AudioJack3_SwitchTR -> Device:R; MPN NMJ6HCD2 -> (none); Spec Neutrik 1/4in stereo jack, horizontal PCB. The footprint's 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 -> 0 ohm, 0603 (ground lift option)
- R44: renamed from RV1; value 10k audio, dual slide -> 100k; footprint (none) -> Resistor_SMD:R_0603_1608Metric; symbol Device:R_Potentiometer_Dual_Separate -> Device:R; MPN PTA2044-2015DPA103 -> (none); Spec Bourns 20 mm travel dual-gang slide pot, 10k audio taper, 1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 -> 1%, 0603
- R45: renamed from U8; value NJM4556AD -> 10; footprint Package_DIP:DIP-8_W7.62mm -> Resistor_SMD:R_0603_1608Metric; symbol Amplifier_Operational:NJM4556A -> Device:R; MPN NJM4556AD -> (none); Spec dual high-current op-amp, DIP-8 -> 1%, 0603
- R46: renamed from C28; value 220uF -> 10k; footprint Capacitor_SMD:CP_Elec_6.3x7.7 -> Resistor_SMD:R_0603_1608Metric; symbol Device:C_Polarized -> Device:R; Spec electrolytic, 10V -> 1%, 0603
- R47: renamed from C32; value 10uF -> 10k; footprint Capacitor_SMD:C_0805_2012Metric -> Resistor_SMD:R_0603_1608Metric; symbol Device:C -> Device:R; Spec X5R, 10V, 0805 -> 1%, 0603
- U6: renamed from C23; value 470pF -> OPA2350UA; footprint Capacitor_SMD:C_0603_1608Metric -> Package_SO:SOIC-8_3.9x4.9mm_P1.27mm; symbol Device:C -> Amplifier_Operational:OPA2340; MPN (none) -> OPA2350UA; Spec C0G, 50V -> dual rail-to-rail op-amp, 2.7-5.5V
- U6: renamed from J4; value 3.5 mm headphones (front) -> OPA2350UA; footprint Connector_Audio:Jack_3.5mm_CUI_SJ1-3523N_Horizontal -> Package_SO:SOIC-8_3.9x4.9mm_P1.27mm; symbol Connector_Audio:AudioJack3 -> Amplifier_Operational:OPA2340; MPN SJ1-3523N -> OPA2350UA; Spec CUI 3.5 mm stereo jack, horizontal -> dual rail-to-rail op-amp, 2.7-5.5V
- U7: renamed from R38; value 10k -> OPA2350UA; footprint Resistor_SMD:R_0603_1608Metric -> Package_SO:SOIC-8_3.9x4.9mm_P1.27mm; symbol Device:R -> Amplifier_Operational:OPA2340; MPN (none) -> OPA2350UA; Spec 1%, 0603 -> dual rail-to-rail op-amp, 2.7-5.5V
- U8: renamed from U7; value OPA2350UA -> NJM4556AD; footprint Package_SO:SOIC-8_3.9x4.9mm_P1.27mm -> Package_DIP:DIP-8_W7.62mm; symbol Amplifier_Operational:OPA2340 -> Amplifier_Operational:NJM4556A; MPN OPA2350UA -> NJM4556AD; Spec dual rail-to-rail op-amp, 2.7-5.5V -> dual high-current op-amp, DIP-8
- U8: renamed from C27; value 1uF -> NJM4556AD; footprint Capacitor_SMD:C_1206_3216Metric -> Package_DIP:DIP-8_W7.62mm; symbol Device:C -> Amplifier_Operational:NJM4556A; MPN (none) -> NJM4556AD; Spec film or X7R 1206, 25V -> dual high-current op-amp, DIP-8
- U8: renamed from R31; value 100k -> NJM4556AD; footprint Resistor_SMD:R_0603_1608Metric -> Package_DIP:DIP-8_W7.62mm; symbol Device:R -> Amplifier_Operational:NJM4556A; MPN (none) -> NJM4556AD; Spec 1%, 0603 -> dual high-current op-amp, DIP-8
- renumbered C29 to C30, C30 to C31, R37 to R38, R47 to R48, U6 to U7
Connections:
- net +4V5A: now also C29.1, U6.8 (V+); no longer C29.8 (V+), R48.1
- net COLD_R: now also C26.1, R36.2, R37.1, R41.1, U6.7; no longer C25.1, C27.1, R37.7, R38.1, U6.2
- net COLD_R_OUT: now also C25.2, J3.R, R42.1; no longer J3.1, R42.2, R43.R
- net COLD_R_R: now also C25.1, R41.2; no longer C25.2, R42.1
- net FR_IN: now also C22.2, R35.1; no longer R35.2, R36.1
- net FR_SUM: now also R35.2, R36.1, U6.6 (-); no longer R36.2, R37.6 (-), U6.1
- net GNDA: now also C29.2, J4.3 (Pin_3), J4.6 (Pin_6), J5.S, R33.2, R40.2, R42.2, R43.2, R46.2, R48.2, U6.4 (V-); no longer C20.3, C22.2, C26.2, C29.4 (V-), J3.2, J5.2, R41.2, R44.6, R47.2, U6.S
- net HOT_R: now also R38.2, R39.1, U7.7; no longer C24.1, R39.7, U7.2
- net HOT_R_OUT: now also C24.2, J3.T, R40.1; no longer R40.2, R41.1, R43.T
- net HOT_R_R: now also C24.1, R39.2; no longer C24.2, R40.1
- net HP_L_DC: now also C21.2, R32.1; no longer R32.2, R34.1
- net HP_L_IN: now also C20.2, U8.3 (+); no longer C21.3 (+), U8.2
- net HP_L_OUT: now also U8.1, U8.2 (-); no longer C21.2 (-), R32.1
- net HP_R_DC: now also C28.2, R45.1, R46.1; no longer J4.1, J5.1, R46.2
- net HP_R_IN: now also C27.2, R44.2, U8.5 (+); no longer C28.2, R45.5 (+), U8.2
- net HP_R_OUT: now also C28.1, U8.6 (-), U8.7; no longer R45.6 (-), R45.7, R46.1
- net INV_R: now also R37.2, R38.1, U7.6 (-); no longer R38.2, R39.6 (-), U7.1
- net PHONE_L: now also J5.T, R32.2; no longer R33.2, U6.T
- net PHONE_R: now also J5.R, R45.2; no longer J4.2, U6.R
- net SLEEVE_R: now also J3.S, R43.1; no longer C26.1, R43.S
- net VOL_L_IN: now also J4.1 (Pin_1); no longer C20.1
- net VOL_L_W: now also C20.1, J4.2 (Pin_2); no longer C20.2, R31.1
- net VOL_R_IN: now also C26.2, J4.4 (Pin_4); no longer C27.2, R44.4
- net VOL_R_W: now also C27.1, J4.5 (Pin_5); no longer R44.5, U8.1
- net VREF: now also R31.1, R44.1, R47.2, R48.1, U6.5 (+), U7.5 (+); no longer C28.1, R37.5 (+), R39.5 (+), R48.2, U8.1
- net YM_MOR: now also R34.1; no longer R35.1
Other:
- moved on the sheet: C30, C31, C32, R33, R34, R36, R38, R41, R48, U7C, U8C

Commit message: Apply the Rev A fix register: decoupling, single ground, A.VCC filter, TPA6132A2
Schematic
- YM2612 A.VCC (pin 22) gets its own 10 ohm + 220 uF + 100 nF filter.
- /IC, A0, A1 pull-downs 10k -> 4.7k (RP2350 erratum E9).
- Headphone amp: NJM4556A replaced by a TPA6132A2 at -6 dB, no output caps,
  enabled by GP12 (HP_EN, 4.7k pull-down) so power-up doesn't pop.
- 47 uF electrolytic damps the L1/C4 resonance before the LP5907.
- GNDA merged into GND; NT1 removed. Four M3 holes for the LCD standoffs.
- Ferrite label 220R@100MHz to match BLM18PG221SN1D; C15/C22 spec X7R 50V;
  LED lead note for PCBWay.
- Pico Plus 2 and its headers marked do-not-fit (Joey supplies them);
  sockets are Sullins PPTC201LFBN-RC.

Layout
- Decoupling caps placed at the pin they serve (design.NEAR), 2-7 mm instead
  of 16-70 mm.
- One solid GND plane on both layers plus 332 stitching vias (tools/stitch.py).
- J6 moved out from under the LCD backpack; encoder moved below the LCD so
  the knob clears it.
- Re-routed with Freerouting; KiCad 7 DRC: 0 errors, 0 unconnected.

Co-Authored-By: Claude Opus 5.5 (1M context) <noreply@anthropic.com>
Claude-Session: https://claude.ai/code/session_01T6y8roX1LzS9uTuKVQBe9X
Parts:
- removed C15: 1uF, Capacitor_SMD:C_1206_3216Metric, symbol Device:C
- removed C16: 470pF, Capacitor_SMD:C_0603_1608Metric, symbol Device:C
- removed R21: 2.2k, Resistor_SMD:R_0603_1608Metric, symbol Device:R
- removed R22: 47k, Resistor_SMD:R_0603_1608Metric, symbol Device:R
- removed R23: 100k, Resistor_SMD:R_0603_1608Metric, symbol Device:R
- removed unit 3 of U6
- removed unit 3 of U7
- added C37: 47uF, Capacitor_SMD:CP_Elec_5x5.4, symbol Device:C_Polarized
- added C38: 100nF, Capacitor_SMD:C_0603_1608Metric, symbol Device:C
- C17: renamed from R24; value 10k -> 1uF; footprint Resistor_SMD:R_0603_1608Metric -> Capacitor_SMD:C_1206_3216Metric; symbol Device:R -> Device:C; Spec 1%, 0603 -> X7R, 50V, 1206
- C18: renamed from R26; value 100 -> 470pF; footprint Resistor_SMD:R_0603_1608Metric -> Capacitor_SMD:C_0603_1608Metric; symbol Device:R -> Device:C; Spec 1%, 0603 -> C0G, 50V
- C19: renamed from J2; value 1/4" TRS balanced out L -> 10uF; footprint Connector_Audio:Jack_6.35mm_Neutrik_NMJ6HCD2_Horizontal -> Capacitor_SMD:CP_Elec_5x5.4; symbol Connector_Audio:AudioJack3_SwitchTR -> Device:C_Polarized; MPN NMJ6HCD2 -> (none); Spec Neutrik 1/4in stereo jack, horizontal PCB. The footprint's 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 -> electrolytic, 16V, low-leakage
- C20: value 1uF -> 10uF; footprint Capacitor_SMD:C_1206_3216Metric -> Capacitor_SMD:CP_Elec_5x5.4; symbol Device:C -> Device:C_Polarized; Spec film or X7R 1206, 25V -> electrolytic, 16V, low-leakage
- C21: renamed from R32; value 10 -> 10uF; footprint Resistor_SMD:R_0603_1608Metric -> Capacitor_SMD:CP_Elec_5x5.4; symbol Device:R -> Device:C_Polarized; Spec 1%, 0603 -> electrolytic, 16V
- C22: renamed from R33; value 10k -> 1uF; footprint Resistor_SMD:R_0603_1608Metric -> Capacitor_SMD:C_1206_3216Metric; symbol Device:R -> Device:C; Spec 1%, 0603 -> X7R, 25V, 1206
- C23: renamed from C22; Spec film or C0G/X7R 1206, 25V (film preferred) -> X7R, 50V, 1206
- C28: renamed from C27; Spec film or X7R 1206, 25V -> X7R, 25V, 1206
- C29: renamed from U8; value NJM4556AD -> 2.2uF; footprint Package_DIP:DIP-8_W7.62mm -> Capacitor_SMD:C_0805_2012Metric; symbol Amplifier_Operational:NJM4556A -> Device:C; MPN NJM4556AD -> (none); Spec dual high-current op-amp, DIP-8 -> X5R, 10V, 0805
- C30: renamed from C28; value 220uF -> 100nF; footprint Capacitor_SMD:CP_Elec_6.3x7.7 -> Capacitor_SMD:C_0603_1608Metric; symbol Device:C_Polarized -> Device:C; Spec electrolytic, 10V -> X7R, 16V
- C31: renamed from R45; value 10 -> 2.2uF; footprint Resistor_SMD:R_0603_1608Metric -> Capacitor_SMD:C_0805_2012Metric; symbol Device:R -> Device:C; Spec 1%, 0603 -> X5R, 10V, 0805
- C32: renamed from R46; value 10k -> 2.2uF; footprint Resistor_SMD:R_0603_1608Metric -> Capacitor_SMD:C_0805_2012Metric; symbol Device:R -> Device:C; Spec 1%, 0603 -> X5R, 10V, 0805
- C33: renamed from J4; value Volume slider (dual 10k audio taper, in the case) -> 1uF; footprint Connector_JST:JST_XH_B6B-XH-A_1x06_P2.50mm_Vertical -> Capacitor_SMD:C_0805_2012Metric; symbol Connector_Generic:Conn_01x06 -> Device:C; MPN B6B-XH-A(LF)(SN) -> (none); Spec JST XH 6-pin header. Wire a dual 10k audio-taper slide pot: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 -> X5R, 10V, 0805 (charge-pump flying cap)
- C34: renamed from C32; value 10uF -> 100nF; footprint Capacitor_SMD:C_0805_2012Metric -> Capacitor_SMD:C_0603_1608Metric; Spec X5R, 10V, 0805 -> X7R, 16V
- C35: renamed from R47; value 10k -> 100nF; footprint Resistor_SMD:R_0603_1608Metric -> Capacitor_SMD:C_0603_1608Metric; symbol Device:R -> Device:C; Spec 1%, 0603 -> X7R, 16V
- C36: renamed from R48; value 10k -> 10uF; footprint Resistor_SMD:R_0603_1608Metric -> Capacitor_SMD:C_0805_2012Metric; symbol Device:R -> Device:C; Spec 1%, 0603 -> X5R, 10V, 0805
- J2: renamed from U8; value NJM4556AD -> 1/4" TRS balanced out L; footprint Package_DIP:DIP-8_W7.62mm -> Connector_Audio:Jack_6.35mm_Neutrik_NMJ6HCD2_Horizontal; symbol Amplifier_Operational:NJM4556A -> Connector_Audio:AudioJack3_SwitchTR; MPN NJM4556AD -> NMJ6HCD2; Spec dual high-current op-amp, DIP-8 -> Neutrik 1/4in stereo jack, horizontal PCB. The footprint's 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
- J4: renamed from U8; value NJM4556AD -> Volume slider (dual 10k audio taper, in the case); footprint Package_DIP:DIP-8_W7.62mm -> Connector_JST:JST_XH_B6B-XH-A_1x06_P2.50mm_Vertical; symbol Amplifier_Operational:NJM4556A -> Connector_Generic:Conn_01x06; MPN NJM4556AD -> B6B-XH-A(LF)(SN); Spec dual high-current op-amp, DIP-8 -> JST XH 6-pin header. Wire a dual 10k audio-taper slide pot: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
- J5: renamed from C29; value 100nF -> 3.5 mm headphones (front); footprint Capacitor_SMD:C_0603_1608Metric -> Connector_Audio:Jack_3.5mm_CUI_SJ1-3523N_Horizontal; symbol Device:C -> Connector_Audio:AudioJack3; MPN (none) -> SJ1-3523N; Spec X7R, 16V -> CUI 3.5 mm stereo jack, horizontal
- R22: renamed from U6; value OPA2350UA -> 2.2k; footprint Package_SO:SOIC-8_3.9x4.9mm_P1.27mm -> Resistor_SMD:R_0603_1608Metric; symbol Amplifier_Operational:OPA2340 -> Device:R; MPN OPA2350UA -> (none); Spec dual rail-to-rail op-amp, 2.7-5.5V -> 1%, 0603
- R23: renamed from R25; value 10k -> 47k
- R24: renamed from U7; value OPA2350UA -> 100k; footprint Package_SO:SOIC-8_3.9x4.9mm_P1.27mm -> Resistor_SMD:R_0603_1608Metric; symbol Amplifier_Operational:OPA2340 -> Device:R; MPN OPA2350UA -> (none); Spec dual rail-to-rail op-amp, 2.7-5.5V -> 1%, 0603
- R25: renamed from R27; value 100k -> 10k
- R26: renamed from R28; value 100 -> 10k
- R27: renamed from R29; value 100k -> 100
- R28: renamed from R30; value 0 -> 100k; Spec 0 ohm, 0603 (ground lift option) -> 1%, 0603
- R29: renamed from C19; value 10uF -> 100; footprint Capacitor_SMD:CP_Elec_5x5.4 -> Resistor_SMD:R_0603_1608Metric; symbol Device:C_Polarized -> Device:R; Spec electrolytic, 16V -> 1%, 0603
- R31: renamed from C21; value 220uF -> 0; footprint Capacitor_SMD:CP_Elec_6.3x7.7 -> Resistor_SMD:R_0603_1608Metric; symbol Device:C_Polarized -> Device:R; Spec electrolytic, 10V -> 0 ohm, 0603 (ground lift option)
- R42: renamed from J5; value 3.5 mm headphones (front) -> 4.7k; footprint Connector_Audio:Jack_3.5mm_CUI_SJ1-3523N_Horizontal -> Resistor_SMD:R_0603_1608Metric; symbol Connector_Audio:AudioJack3 -> Device:R; MPN SJ1-3523N -> (none); Spec CUI 3.5 mm stereo jack, horizontal -> 1%, 0603
- R43: renamed from C33; value 47uF -> 10k; footprint Capacitor_SMD:CP_Elec_5x5.4 -> Resistor_SMD:R_0603_1608Metric; symbol Device:C_Polarized -> Device:R; Spec electrolytic, 16V -> 1%, 0603
- R44: renamed from C34; value 100nF -> 10k; footprint Capacitor_SMD:C_0603_1608Metric -> Resistor_SMD:R_0603_1608Metric; symbol Device:C -> Device:R; Spec X7R, 16V -> 1%, 0603
- U6: renamed from C30; value 100nF -> OPA2350UA; footprint Capacitor_SMD:C_0603_1608Metric -> Package_SO:SOIC-8_3.9x4.9mm_P1.27mm; symbol Device:C -> Amplifier_Operational:OPA2340; MPN (none) -> OPA2350UA; Spec X7R, 16V -> dual rail-to-rail op-amp, 2.7-5.5V
- U6: renamed from C17; value 10uF -> OPA2350UA; footprint Capacitor_SMD:CP_Elec_5x5.4 -> Package_SO:SOIC-8_3.9x4.9mm_P1.27mm; symbol Device:C_Polarized -> Amplifier_Operational:OPA2340; MPN (none) -> OPA2350UA; Spec electrolytic, 16V, low-leakage -> dual rail-to-rail op-amp, 2.7-5.5V
- U7: renamed from C31; value 100nF -> OPA2350UA; footprint Capacitor_SMD:C_0603_1608Metric -> Package_SO:SOIC-8_3.9x4.9mm_P1.27mm; symbol Device:C -> Amplifier_Operational:OPA2340; MPN (none) -> OPA2350UA; Spec X7R, 16V -> dual rail-to-rail op-amp, 2.7-5.5V
- U7: renamed from C18; value 10uF -> OPA2350UA; footprint Capacitor_SMD:CP_Elec_5x5.4 -> Package_SO:SOIC-8_3.9x4.9mm_P1.27mm; symbol Device:C_Polarized -> Amplifier_Operational:OPA2340; MPN (none) -> OPA2350UA; Spec electrolytic, 16V, low-leakage -> dual rail-to-rail op-amp, 2.7-5.5V
- U8: renamed from R44; value 100k -> TPA6132A2RTER; footprint Resistor_SMD:R_0603_1608Metric -> Package_DFN_QFN:WQFN-16-1EP_3x3mm_P0.5mm_EP1.68x1.68mm; symbol Device:R -> Amplifier_Audio:TPA6132A2RTE; MPN (none) -> TPA6132A2RTER; Spec 1%, 0603 -> TI DirectPath stereo headphone amp, 2.3-5.5V, WQFN-16 3x3 m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
- renumbered C23 to C24, C24 to C25, C25 to C26, C26 to C27, R31 to R30, R34 to R32, R35 to R33, R36 to R34, R37 to R35, R38 to R36, R39 to R37, R40 to R38, R41 to R39, R42 to R40, R43 to R41
Connections:
- net +4V5A: now also C29.1, C30.1, C36.1, R43.1, U6.8 (V+), U7.8 (V+), U8.14 (VDD); no longer J4.8 (V+), J5.1, U6.1, U7.1
- net COLD_L: now also C18.2, C21.1, R24.2, R25.1, U6.1; no longer C17.1, R22.1, R26.1
- net COLD_L_OUT: now also C20.2, J2.R, R30.1; no longer C19.R, R27.1, U7.2
- net COLD_L_R: now also C20.1, R29.2; no longer R26.2, U7.1
- net FL_IN: now also C17.2, R23.1
- net FL_SUM: now also C18.1, R23.2, R24.1, U6.2 (-); no longer R22.2 (-)
- net HOT_L: now also R26.2, R27.1, U7.1; no longer C18.1, R23.2, R24.1
- net HOT_L_OUT: now also C19.2, J2.T, R28.1; no longer C19.T, R25.1, U6.2
- net HOT_L_R: now also C19.1, R27.2; no longer C18.2, U6.1
- net HP_L_IN: now also C22.2, U8.1 (INL-); no longer C20.2, J2.3 (+), R30.2
- net HP_R_IN: now also U8.4 (INR-); no longer C29.5 (+), U8.2
- net INV_L: now also R25.2, R26.1, U7.2 (-); no longer C17.2, R23.1, R24.2 (-)
- net PHONE_L: now also J5.T, U8.16 (OUTL); no longer C21.2, R42.T
- net PHONE_R: now also J5.R, U8.5 (OUTR); no longer C31.2, R42.R
- net SLEEVE_L: now also J2.S, R31.1; no longer C19.S, R28.1
- net VOL_L_IN: now also C21.2, J4.1 (Pin_1); no longer C33.1 (Pin_1), R29.2
- net VOL_L_W: now also C22.1, J4.2 (Pin_2); no longer C20.1, C33.2 (Pin_2)
- net VOL_R_IN: now also J4.4 (Pin_4); no longer C33.4 (Pin_4)
- net VOL_R_W: now also J4.5 (Pin_5); no longer C33.5 (Pin_5)
- net VREF: now also R43.2, U6.3 (+), U7.3 (+), C37.1, C38.1; no longer C35.2, C36.1, R22.3 (+), R24.3 (+), R30.1, R43.1, U8.1
- net YM_MOL: now also C17.1, R22.1
- removed net GNDA: C22.2, C32.2, C33.3 (Pin_3), C33.6 (Pin_6), C34.2, C36.2, J4.4 (V-), J5.2, R25.2, R27.2, R28.2, R32.2, R38.2, R40.2, R41.2, R42.S, R43.2, R44.2, U6.2, U7.2
- removed net HP_L_DC: C21.1, C22.1, R31.2
- removed net HP_L_OUT: J2.1, J2.2 (-), R31.1
- removed net HP_R_DC: C30.2, C31.1, C32.1
- removed net HP_R_OUT: C29.6 (-), C29.7, C30.1
- new net GND: C29.2, C30.2, C31.2, C32.2, C34.2, C35.2, C36.2, C37.2, C38.2, J4.3 (Pin_3), J4.6 (Pin_6), J5.S, R22.2, R28.2, R30.2, R31.2, R32.2, R38.2, R40.2, R41.2, R42.2, R44.2, U6.4 (V-), U7.4 (V-), U8.10 (PGND), U8.15 (SGND), U8.17 (EP), U8.2 (INL+), U8.3 (INR+), U8.6 (G0), U8.7 (G1)
- new net HPVDD: C31.1, U8.12 (HPVDD)
- new net HPVSS: C32.1, U8.8 (HPVSS)
- new net HP_CPN: C33.2, U8.9 (CPN)
- new net HP_CPP: C33.1, U8.11 (CPP)
- new net HP_EN: R42.1, U8.13 (EN)
Other:
- note added: "AUDIO OUT (authentic Model 1 sound, no clean mode). Everything here runs on the quiet +4V5A rail around VREF = 2.25V. 1. 2.2k load on MOL / MOR, as in the Mega Amp, so the chip's DAC works as it did in the console. 2. Model 1 style low-pass: inverting OPA2350 stage, 47k in, 100k || 470pF feedback. First order, 3.39 kHz, gain about 2.1. That matches the 47k / 1nF Model 1 filter used by MIDIbox. Ch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"
- note removed: "AUDIO OUT (authentic Model 1 sound, no clean mode). Everything here runs on the quiet +4V5A rail around VREF = 2.25V, grounded to GNDA. 1. 2.2k load on MOL / MOR, as in the Mega Amp, so the chip's DAC works as it did in the console. 2. Model 1 style low-pass: inverting OPA2350 stage, 47k in, 100k || 470pF feedback. First order, 3.39 kHz, gain about 2.1. That matches the 47k / 1nF Model 1 filter u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"
- moved on the sheet: C34, R23, R25, R26, R27, R28, R30

Commit message: Schematic: draw real wires between parts instead of name tags
tools/wires.py routes each page's nets on the 1.27 mm grid around part bodies and text.
Power pins keep power symbols (neighbouring pins share one), signals that leave a page get
one global label, and the netlist check still matches design.py exactly (0 mismatches).
Sound chip and audio pages re-laid out so the wiring reads left to right; title blocks say Rev B.

Co-Authored-By: Claude Opus 5.5 <noreply@anthropic.com>
Claude-Session: https://claude.ai/code/session_01TDTDVidYRoyJdUGgsyVTSw
Other:
- moved on the sheet: C21, C22, C27, C28, C29, C30, C31, C32, C33, J4, J5, R42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

Commit message: Schematic: PWR_FLAG on YM_AVCC (KiCad 10 ERC: A.VCC is fed through R21)
Co-Authored-By: Claude Opus 5.5 <noreply@anthropic.com>
Claude-Session: https://claude.ai/code/session_01TDTDVidYRoyJdUGgsyVTSw
Parts:
- removed J4: Volume slider (dual 10k audio taper, in the case), Connector_JST:JST_XH_B6B-XH-A_1x06_P2.50mm_Vertical, symbol Connector_Generic:Conn_01x06
- removed R22: 2.2k, Resistor_SMD:R_0603_1608Metric, symbol Device:R
- added C38: 100nF, Capacitor_SMD:C_0603_1608Metric, symbol Device:C
- added R42: 4.7k, Resistor_SMD:R_0603_1608Metric, symbol Device:R
- C17: renamed from R23; value 47k -> 1uF; footprint Resistor_SMD:R_0603_1608Metric -> Capacitor_SMD:C_1206_3216Metric; symbol Device:R -> Device:C; Spec 1%, 0603 -> X7R, 50V, 1206
- C18, C24: renamed from U6; value OPA2350UA -> 470pF; footprint Package_SO:SOIC-8_3.9x4.9mm_P1.27mm -> Capacitor_SMD:C_0603_1608Metric; symbol Amplifier_Operational:OPA2340 -> Device:C; MPN OPA2350UA -> (none); Spec dual rail-to-rail op-amp, 2.7-5.5V -> C0G, 50V
- C19: renamed from R28; value 100k -> 10uF; footprint Resistor_SMD:R_0603_1608Metric -> Capacitor_SMD:CP_Elec_5x5.4; symbol Device:R -> Device:C_Polarized; Spec 1%, 0603 -> electrolytic, 16V, low-leakage
- C20: renamed from R30; value 100k -> 10uF; footprint Resistor_SMD:R_0603_1608Metric -> Capacitor_SMD:CP_Elec_5x5.4; symbol Device:R -> Device:C_Polarized; Spec 1%, 0603 -> electrolytic, 16V, low-leakage
- C21: renamed from C22; value 1uF -> 10uF; footprint Capacitor_SMD:C_1206_3216Metric -> Capacitor_SMD:CP_Elec_5x5.4; symbol Device:C -> Device:C_Polarized; Spec X7R, 25V, 1206 -> electrolytic, 16V
- C22: renamed from R32; value 2.2k -> 1uF; footprint Resistor_SMD:R_0603_1608Metric -> Capacitor_SMD:C_1206_3216Metric; symbol Device:R -> Device:C; Spec 1%, 0603 -> X7R, 25V, 1206
- C23: renamed from R33; value 47k -> 1uF; footprint Resistor_SMD:R_0603_1608Metric -> Capacitor_SMD:C_1206_3216Metric; symbol Device:R -> Device:C; Spec 1%, 0603 -> X7R, 50V, 1206
- C25: renamed from R38; value 100k -> 10uF; footprint Resistor_SMD:R_0603_1608Metric -> Capacitor_SMD:CP_Elec_5x5.4; symbol Device:R -> Device:C_Polarized; Spec 1%, 0603 -> electrolytic, 16V, low-leakage
- C26: renamed from R40; value 100k -> 10uF; footprint Resistor_SMD:R_0603_1608Metric -> Capacitor_SMD:CP_Elec_5x5.4; symbol Device:R -> Device:C_Polarized; Spec 1%, 0603 -> electrolytic, 16V, low-leakage
- C27: renamed from C28; value 1uF -> 10uF; footprint Capacitor_SMD:C_1206_3216Metric -> Capacitor_SMD:CP_Elec_5x5.4; symbol Device:C -> Device:C_Polarized; Spec X7R, 25V, 1206 -> electrolytic, 16V
- C28: renamed from U8; value TPA6132A2RTER -> 1uF; footprint Package_DFN_QFN:WQFN-16-1EP_3x3mm_P0.5mm_EP1.68x1.68mm -> Capacitor_SMD:C_1206_3216Metric; symbol Amplifier_Audio:TPA6132A2RTE -> Device:C; MPN TPA6132A2RTER -> (none); Spec TI DirectPath stereo headphone amp, 2.3-5.5V, WQFN-16 3x3 m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 -> X7R, 25V, 1206
- C29: renamed from C30; value 100nF -> 2.2uF; footprint Capacitor_SMD:C_0603_1608Metric -> Capacitor_SMD:C_0805_2012Metric; Spec X7R, 16V -> X5R, 10V, 0805
- C30: renamed from C31; value 2.2uF -> 100nF; footprint Capacitor_SMD:C_0805_2012Metric -> Capacitor_SMD:C_0603_1608Metric; Spec X5R, 10V, 0805 -> X7R, 16V
- C32: renamed from C33; value 1uF -> 2.2uF; Spec X5R, 10V, 0805 (charge-pump flying cap) -> X5R, 10V, 0805
- C33: renamed from R42; value 4.7k -> 1uF; footprint Resistor_SMD:R_0603_1608Metric -> Capacitor_SMD:C_0805_2012Metric; symbol Device:R -> Device:C; Spec 1%, 0603 -> X5R, 10V, 0805 (charge-pump flying cap)
- C35: renamed from C36; value 10uF -> 100nF; footprint Capacitor_SMD:C_0805_2012Metric -> Capacitor_SMD:C_0603_1608Metric; Spec X5R, 10V, 0805 -> X7R, 16V
- C36: renamed from R43; value 10k -> 10uF; footprint Resistor_SMD:R_0603_1608Metric -> Capacitor_SMD:C_0805_2012Metric; symbol Device:R -> Device:C; Spec 1%, 0603 -> X5R, 10V, 0805
- C37: renamed from C38; value 100nF -> 47uF; footprint Capacitor_SMD:C_0603_1608Metric -> Capacitor_SMD:CP_Elec_5x5.4; symbol Device:C -> Device:C_Polarized; Spec X7R, 16V -> electrolytic, 16V
- J2: renamed from R31; value 0 -> 1/4" TRS balanced out L; footprint Resistor_SMD:R_0603_1608Metric -> Connector_Audio:Jack_6.35mm_Neutrik_NMJ6HCD2_Horizontal; symbol Device:R -> Connector_Audio:AudioJack3_SwitchTR; MPN (none) -> NMJ6HCD2; Spec 0 ohm, 0603 (ground lift option) -> Neutrik 1/4in stereo jack, horizontal PCB. The footprint's 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
- J3: renamed from R41; value 0 -> 1/4" TRS balanced out R; footprint Resistor_SMD:R_0603_1608Metric -> Connector_Audio:Jack_6.35mm_Neutrik_NMJ6HCD2_Horizontal; symbol Device:R -> Connector_Audio:AudioJack3_SwitchTR; MPN (none) -> NMJ6HCD2; Spec 0 ohm, 0603 (ground lift option) -> Neutrik 1/4in stereo jack, horizontal PCB. The footprint's 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
- J4: renamed from J5; value 3.5 mm headphones (front) -> Volume slider (dual 10k audio taper, in the case); footprint Connector_Audio:Jack_3.5mm_CUI_SJ1-3523N_Horizontal -> Connector_JST:JST_XH_B6B-XH-A_1x06_P2.50mm_Vertical; symbol Connector_Audio:AudioJack3 -> Connector_Generic:Conn_01x06; MPN SJ1-3523N -> B6B-XH-A(LF)(SN); Spec CUI 3.5 mm stereo jack, horizontal -> JST XH 6-pin header. Wire a dual 10k audio-taper slide pot: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
- J5: renamed from U6; value OPA2350UA -> 3.5 mm headphones (front); footprint Package_SO:SOIC-8_3.9x4.9mm_P1.27mm -> Connector_Audio:Jack_3.5mm_CUI_SJ1-3523N_Horizontal; symbol Amplifier_Operational:OPA2340 -> Connector_Audio:AudioJack3; MPN OPA2350UA -> SJ1-3523N; Spec dual rail-to-rail op-amp, 2.7-5.5V -> CUI 3.5 mm stereo jack, horizontal
- R22: renamed from C17; value 1uF -> 2.2k; footprint Capacitor_SMD:C_1206_3216Metric -> Resistor_SMD:R_0603_1608Metric; symbol Device:C -> Device:R; Spec X7R, 50V, 1206 -> 1%, 0603
- R23: renamed from R24; value 100k -> 47k
- R24: renamed from C18; value 470pF -> 100k; footprint Capacitor_SMD:C_0603_1608Metric -> Resistor_SMD:R_0603_1608Metric; symbol Device:C -> Device:R; Spec C0G, 50V -> 1%, 0603
- R26, R36: renamed from U7; value OPA2350UA -> 10k; footprint Package_SO:SOIC-8_3.9x4.9mm_P1.27mm -> Resistor_SMD:R_0603_1608Metric; symbol Amplifier_Operational:OPA2340 -> Device:R; MPN OPA2350UA -> (none); Spec dual rail-to-rail op-amp, 2.7-5.5V -> 1%, 0603
- R27: renamed from C19; value 10uF -> 100; footprint Capacitor_SMD:CP_Elec_5x5.4 -> Resistor_SMD:R_0603_1608Metric; symbol Device:C_Polarized -> Device:R; Spec electrolytic, 16V, low-leakage -> 1%, 0603
- R28: renamed from R29; value 100 -> 100k
- R29: renamed from C20; value 10uF -> 100; footprint Capacitor_SMD:CP_Elec_5x5.4 -> Resistor_SMD:R_0603_1608Metric; symbol Device:C_Polarized -> Device:R; Spec electrolytic, 16V, low-leakage -> 1%, 0603
- R30: renamed from J2; value 1/4" TRS balanced out L -> 100k; footprint Connector_Audio:Jack_6.35mm_Neutrik_NMJ6HCD2_Horizontal -> Resistor_SMD:R_0603_1608Metric; symbol Connector_Audio:AudioJack3_SwitchTR -> Device:R; MPN NMJ6HCD2 -> (none); Spec Neutrik 1/4in stereo jack, horizontal PCB. The footprint's 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 -> 1%, 0603
- R31: renamed from C21; value 10uF -> 0; footprint Capacitor_SMD:CP_Elec_5x5.4 -> Resistor_SMD:R_0603_1608Metric; symbol Device:C_Polarized -> Device:R; Spec electrolytic, 16V -> 0 ohm, 0603 (ground lift option)
- R32: renamed from C23; value 1uF -> 2.2k; footprint Capacitor_SMD:C_1206_3216Metric -> Resistor_SMD:R_0603_1608Metric; symbol Device:C -> Device:R; Spec X7R, 50V, 1206 -> 1%, 0603
- R33: renamed from R34; value 100k -> 47k
- R34: renamed from C24; value 470pF -> 100k; footprint Capacitor_SMD:C_0603_1608Metric -> Resistor_SMD:R_0603_1608Metric; symbol Device:C -> Device:R; Spec C0G, 50V -> 1%, 0603
- R37: renamed from C25; value 10uF -> 100; footprint Capacitor_SMD:CP_Elec_5x5.4 -> Resistor_SMD:R_0603_1608Metric; symbol Device:C_Polarized -> Device:R; Spec electrolytic, 16V, low-leakage -> 1%, 0603
- R38: renamed from R39; value 100 -> 100k
- R39: renamed from C26; value 10uF -> 100; footprint Capacitor_SMD:CP_Elec_5x5.4 -> Resistor_SMD:R_0603_1608Metric; symbol Device:C_Polarized -> Device:R; Spec electrolytic, 16V, low-leakage -> 1%, 0603
- R40: renamed from J3; value 1/4" TRS balanced out R -> 100k; footprint Connector_Audio:Jack_6.35mm_Neutrik_NMJ6HCD2_Horizontal -> Resistor_SMD:R_0603_1608Metric; symbol Connector_Audio:AudioJack3_SwitchTR -> Device:R; MPN NMJ6HCD2 -> (none); Spec Neutrik 1/4in stereo jack, horizontal PCB. The footprint's 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 -> 1%, 0603
- R41: renamed from C27; value 10uF -> 0; footprint Capacitor_SMD:CP_Elec_5x5.4 -> Resistor_SMD:R_0603_1608Metric; symbol Device:C_Polarized -> Device:R; Spec electrolytic, 16V -> 0 ohm, 0603 (ground lift option)
- R44: renamed from C37; value 47uF -> 10k; footprint Capacitor_SMD:CP_Elec_5x5.4 -> Resistor_SMD:R_0603_1608Metric; symbol Device:C_Polarized -> Device:R; Spec electrolytic, 16V -> 1%, 0603
- U6: renamed from R25; value 10k -> OPA2350UA; footprint Resistor_SMD:R_0603_1608Metric -> Package_SO:SOIC-8_3.9x4.9mm_P1.27mm; symbol Device:R -> Amplifier_Operational:OPA2340; MPN (none) -> OPA2350UA; Spec 1%, 0603 -> dual rail-to-rail op-amp, 2.7-5.5V
- U6: renamed from R35; value 10k -> OPA2350UA; footprint Resistor_SMD:R_0603_1608Metric -> Package_SO:SOIC-8_3.9x4.9mm_P1.27mm; symbol Device:R -> Amplifier_Operational:OPA2340; MPN (none) -> OPA2350UA; Spec 1%, 0603 -> dual rail-to-rail op-amp, 2.7-5.5V
- U7: renamed from R27; value 100 -> OPA2350UA; footprint Resistor_SMD:R_0603_1608Metric -> Package_SO:SOIC-8_3.9x4.9mm_P1.27mm; symbol Device:R -> Amplifier_Operational:OPA2340; MPN (none) -> OPA2350UA; Spec 1%, 0603 -> dual rail-to-rail op-amp, 2.7-5.5V
- U7: renamed from R37; value 100 -> OPA2350UA; footprint Resistor_SMD:R_0603_1608Metric -> Package_SO:SOIC-8_3.9x4.9mm_P1.27mm; symbol Device:R -> Amplifier_Operational:OPA2340; MPN (none) -> OPA2350UA; Spec 1%, 0603 -> dual rail-to-rail op-amp, 2.7-5.5V
- U7: renamed from C34; value 100nF -> OPA2350UA; footprint Capacitor_SMD:C_0603_1608Metric -> Package_SO:SOIC-8_3.9x4.9mm_P1.27mm; symbol Device:C -> Amplifier_Operational:OPA2340; MPN (none) -> OPA2350UA; Spec X7R, 16V -> dual rail-to-rail op-amp, 2.7-5.5V
- U8: renamed from C29; value 2.2uF -> TPA6132A2RTER; footprint Capacitor_SMD:C_0805_2012Metric -> Package_DFN_QFN:WQFN-16-1EP_3x3mm_P0.5mm_EP1.68x1.68mm; symbol Device:C -> Amplifier_Audio:TPA6132A2RTE; MPN (none) -> TPA6132A2RTER; Spec X5R, 10V, 0805 -> TI DirectPath stereo headphone amp, 2.3-5.5V, WQFN-16 3x3 m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
- renumbered C32 to C31, C35 to C34, R26 to R25, R36 to R35, R44 to R43, U7 to U6
Connections:
- net +4V5A: now also C30.1, R43.1, U7.8 (V+), U8.14 (VDD); no longer C28.14 (VDD), J5.8 (V+), U7.1, U8.1
- net COLD_L: now also C18.2, C21.1, R25.1, R29.1; no longer C18.1, R23.2, R28.1, R31.1
- net COLD_L_OUT: now also C20.2, J2.R, R30.1; no longer C20.1, R29.2, R30.R
- net COLD_L_R: now also C20.1, R29.2; no longer R28.2, R29.1
- net COLD_R: now also C24.2, C27.1, R35.1, R39.1, U6.7; no longer C24.7, R33.2, R38.1, R41.1, U6.1
- net COLD_R_OUT: now also C26.2, J3.R, R40.1; no longer C26.1, R39.2, R40.R
- net COLD_R_R: now also C26.1, R39.2; no longer R38.2, R39.1
- net FL_IN: now also C17.2, R23.1; no longer C17.1, R22.2
- net FL_SUM: now also C18.1, R23.2, U6.2 (-); no longer C17.2, C18.2 (-), R23.1
- net FR_IN: now also C23.2, R33.1; no longer C23.1, R32.2
- net FR_SUM: now also C24.1, R33.2, U6.6 (-); no longer C23.2, C24.6 (-), R33.1
- net GND: now also C32.2, C36.2, J4.3 (Pin_3), J4.6 (Pin_6), J5.S, R22.2, R28.2, R30.2, R31.2, R32.2, R38.2, R40.2, R41.2, U7.4 (V-), U8.10 (PGND), U8.15 (SGND), U8.17 (EP), U8.3 (INR+), U8.6 (G0), U8.7 (G1), C38.2, R42.2; no longer C19.2, C20.2, C22.2, C25.2, C26.2, C28.10 (PGND), C28.15 (SGND), C28.17 (EP), C28.2 (INL+), C28.3 (INR+), C28.6 (G0), C28.7 (G1), C33.2, J2.2, J3.2, J4.S, J5.4 (V-), R43.2, U7.2
- net HOT_L: now also R26.2, R27.1; no longer R25.2, R26.1
- net HOT_L_OUT: now also C19.2, J2.T, R28.1; no longer C19.1, R27.2, R30.T
- net HOT_L_R: now also C19.1, R27.2; no longer R27.1, U7.2
- net HOT_R: now also R36.2, R37.1, U7.7; no longer R35.2, R36.7, U7.1
- net HOT_R_OUT: now also C25.2, J3.T, R38.1; no longer C25.1, R37.2, R40.T
- net HOT_R_R: now also C25.1, R37.2; no longer R37.1, U7.2
- net HPVDD: now also C31.1, U8.12 (HPVDD); no longer C28.12 (HPVDD), C30.1
- net HPVSS: now also C32.1, U8.8 (HPVSS); no longer C28.8 (HPVSS), C31.1
- net HP_CPN: now also C33.2, U8.9 (CPN); no longer C28.9 (CPN), C32.2
- net HP_CPP: now also C33.1, U8.11 (CPP); no longer C28.11 (CPP), C32.1
- net HP_EN: now also U8.13 (EN), R42.1; no longer C28.13 (EN), C33.1
- net HP_L_IN: now also C22.2, U8.1 (INL-); no longer C21.2, C28.1 (INL-)
- net HP_R_IN: now also C28.2, U8.4 (INR-); no longer C27.2, C28.4 (INR-)
- net INV_L: now also R25.2, R26.1, U7.2 (-); no longer R25.1, R26.2 (-), U6.2
- net INV_R: now also R35.2, R36.1, U7.6 (-); no longer R35.1, R36.6 (-), U6.2
- net PHONE_L: now also J5.T, U8.16 (OUTL); no longer C28.16 (OUTL), J4.T
- net PHONE_R: now also J5.R, U8.5 (OUTR); no longer C28.5 (OUTR), J4.R
- net SLEEVE_L: now also J2.S, R31.1; no longer J2.1, R30.S
- net SLEEVE_R: now also J3.S, R41.1; no longer J3.1, R40.S
- net VOL_L_IN: now also C21.2, J4.1 (Pin_1); no longer R31.2
- net VOL_L_W: now also C22.1, J4.2 (Pin_2); no longer C21.1
- net VOL_R_IN: now also C27.2, J4.4 (Pin_4); no longer R41.2
- net VOL_R_W: now also C28.1, J4.5 (Pin_5); no longer C27.1
- net VREF: now also R43.2, U6.3 (+), U6.5 (+), U7.3 (+), U7.5 (+), C38.1; no longer C18.3 (+), C24.5 (+), C36.2, R26.3 (+), R36.5 (+), R43.1
- net YM_MOL: now also C17.1
- net YM_MOR: now also C23.1; no longer C22.1
Other:
- moved on the sheet: C29, C30, C31, C32, C34, C35, R23, R25, R28, R33, R35, R38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
