File: hardware/ym2612_player/ym2612_player.kicad_pcb (KiCad board)
At the start: 2 copper layers, 240 x 120 mm, 142 parts, among them J1 Spare GPIO (not fitted), J2 1/4" TRS balanced out L, J3 1/4" TRS balanced out R, J4 Volume slider (dual 10k audio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, J5 3.5 mm headphones (front), J6 LCD (I2C backpack: GND, VCC, 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, Q1 BSS138, Q2 BSS138, SW1 Play (red cap), SW2 Stop, SW3 Left, SW4 Right, SW5 Edit, SW6 Exit, SW7 Write, SW8 Data knob, U1 LP5907MFX-4.5, U2 Pimoroni Pico Plus 2, U3 74HCT541, U4 74HCT541, U5 YM2612 (socket only, chip fit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, U6 OPA2350UA, U7 OPA2350UA, U8 NJM4556AD, X1 7.670454 MHz, 5V (not fitted)

Commit message: Mount the Pico Plus 2 on sockets, pick the window LED, tidy labels
The Pico Plus 2 has flash, PSRAM and a connector on its underside, so it
can't be soldered flat. It now plugs into two 1x20 female sockets in the
standard Pico hole pattern; the BOM gains the sockets and the headers for
the module. Tracks around it are re-routed. DRC in KiCad 10: 0 errors,
0 unconnected, matches the schematic.

Window LEDs: Lumimax LED3WAW (3 mm warm white). New tools/silk.py moves
part labels clear of pads and each other; values move to the fab layer.

Co-Authored-By: Claude Opus 5.5 (1M context) <noreply@anthropic.com>
Claude-Session: https://claude.ai/code/session_01JeM5NcWqyQVA3DixJkw6Wg
Parts:
- U2: footprint ym2612:Pimoroni_PicoPlus2_SMD -> ym2612:Pimoroni_PicoPlus2_Socketed
Routing:
- net GNDA: track 361.4 -> 387.8 mm
- net I2C_SCL: track 59.0 -> 44.6 mm, vias 2 -> 1
- net GND: track 691.1 -> 700.4 mm
- net MCU_D4: track 31.7 -> 22.8 mm, vias 2 -> 1
- net MCU_D0: track 45.4 -> 39.8 mm
- net MCU_D3: track 22.3 -> 27.9 mm
- net MCU_D1: track 35.4 -> 30.3 mm
- net +3V3: track 190.8 -> 187.4 mm
- net MCU_D6: track 17.2 -> 20.3 mm, vias 2 -> 1
- net +5V: track 241.6 -> 238.5 mm, vias 5 -> 6
- net MCU_A0: track 46.0 -> 43.0 mm
- net MCU_D7: track 27.5 -> 24.7 mm
- net MCU_D5: track 20.0 -> 22.2 mm
- net HP_L_OUT: track 9.07 -> 11.3 mm
- net YM_CLK: track 21.1 -> 23.2 mm
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
Commit message: Apply the Rev A fix register: decoupling, single ground, A.VCC filter, TPA6132A2
Schematic
- YM2612 A.VCC (pin 22) gets its own 10 ohm + 220 uF + 100 nF filter.
- /IC, A0, A1 pull-downs 10k -> 4.7k (RP2350 erratum E9).
- Headphone amp: NJM4556A replaced by a TPA6132A2 at -6 dB, no output caps,
  enabled by GP12 (HP_EN, 4.7k pull-down) so power-up doesn't pop.
- 47 uF electrolytic damps the L1/C4 resonance before the LP5907.
- GNDA merged into GND; NT1 removed. Four M3 holes for the LCD standoffs.
- Ferrite label 220R@100MHz to match BLM18PG221SN1D; C15/C22 spec X7R 50V;
  LED lead note for PCBWay.
- Pico Plus 2 and its headers marked do-not-fit (Joey supplies them);
  sockets are Sullins PPTC201LFBN-RC.

Layout
- Decoupling caps placed at the pin they serve (design.NEAR), 2-7 mm instead
  of 16-70 mm.
- One solid GND plane on both layers plus 332 stitching vias (tools/stitch.py).
- J6 moved out from under the LCD backpack; encoder moved below the LCD so
  the knob clears it.
- Re-routed with Freerouting; KiCad 7 DRC: 0 errors, 0 unconnected.

Co-Authored-By: Claude Opus 5.5 (1M context) <noreply@anthropic.com>
Claude-Session: https://claude.ai/code/session_01T6y8roX1LzS9uTuKVQBe9X
Parts:
- removed NT1: GND-GNDA join, NetTie:NetTie-2_SMD_Pad2.0mm
- removed R51, R52, R53, R54: 4.7k, Resistor_SMD:R_0603_1608Metric
- added C39: 10nF, Capacitor_SMD:C_0603_1608Metric, F.Cu at (218.2, 99.6)
- added C40: 10nF, Capacitor_SMD:C_0603_1608Metric, F.Cu at (218.8, 101.5)
- added C41: 10uF, Capacitor_SMD:C_0805_2012Metric, F.Cu at (175.6, 65.5)
- added C42: 100nF, Capacitor_SMD:C_0603_1608Metric, F.Cu at (171.4, 53.6)
- added H5: M3 (LCD), MountingHole:MountingHole_3.2mm_M3, F.Cu at (176.5, 60.5)
- added H6: M3 (LCD), MountingHole:MountingHole_3.2mm_M3, F.Cu at (269.5, 60.5)
- added H7: M3 (LCD), MountingHole:MountingHole_3.2mm_M3, F.Cu at (176.5, 115.5)
- added H8: M3 (LCD), MountingHole:MountingHole_3.2mm_M3, F.Cu at (269.5, 115.5)
- C15: value 1uF -> 220uF; footprint Capacitor_SMD:C_1206_3216Metric -> Capacitor_SMD:CP_Elec_6.3x7.7
- C16: value 470pF -> 100nF
- C17: value 10uF -> 1uF; footprint Capacitor_SMD:CP_Elec_5x5.4 -> Capacitor_SMD:C_1206_3216Metric
- C18, C24: value 10uF -> 470pF; footprint Capacitor_SMD:CP_Elec_5x5.4 -> Capacitor_SMD:C_0603_1608Metric
- C20, C27: value 1uF -> 10uF; footprint Capacitor_SMD:C_1206_3216Metric -> Capacitor_SMD:CP_Elec_5x5.4
- C21: value 220uF -> 10uF; footprint Capacitor_SMD:CP_Elec_6.3x7.7 -> Capacitor_SMD:CP_Elec_5x5.4
- C23: value 470pF -> 1uF; footprint Capacitor_SMD:C_0603_1608Metric -> Capacitor_SMD:C_1206_3216Metric
- C28: value 220uF -> 1uF; footprint Capacitor_SMD:CP_Elec_6.3x7.7 -> Capacitor_SMD:C_1206_3216Metric
- C29, C31: value 100nF -> 2.2uF; footprint Capacitor_SMD:C_0603_1608Metric -> Capacitor_SMD:C_0805_2012Metric
- C32: value 10uF -> 2.2uF
- C33: value 47uF -> 1uF; footprint Capacitor_SMD:CP_Elec_5x5.4 -> Capacitor_SMD:C_0805_2012Metric
- C35: value 10nF -> 100nF
- C36: value 10nF -> 10uF; footprint Capacitor_SMD:C_0603_1608Metric -> Capacitor_SMD:C_0805_2012Metric
- C37, C7: value 10uF -> 47uF; footprint Capacitor_SMD:C_0805_2012Metric -> Capacitor_SMD:CP_Elec_5x5.4
- C5: value 4.7uF -> 47uF; footprint Capacitor_SMD:C_0805_2012Metric -> Capacitor_SMD:CP_Elec_5x5.4
- C6: value 47uF -> 4.7uF; footprint Capacitor_SMD:CP_Elec_5x5.4 -> Capacitor_SMD:C_0805_2012Metric
- C8: value 100nF -> 10uF; footprint Capacitor_SMD:C_0603_1608Metric -> Capacitor_SMD:C_0805_2012Metric
- FB1, FB2: value 600R@100MHz -> 220R@100MHz
- R2, R3, R4, R47, R48, R49, R50: value 10k -> 4.7k
- R21: value 2.2k -> 10
- R22: value 47k -> 2.2k
- R23: value 100k -> 47k
- R24, R38: value 10k -> 100k
- R26: value 100 -> 10k
- R27, R29: value 100k -> 100
- R28: value 100 -> 100k
- R30: value 0 -> 100k
- R31: value 100k -> 0
- R32: value 10 -> 2.2k
- R33: value 10k -> 47k
- R34: value 2.2k -> 100k
- R35: value 47k -> 10k
- R36, R44: value 100k -> 10k
- R37: value 10k -> 100
- R41: value 100 -> 0
- R42: value 100k -> 4.7k
- R43: value 0 -> 10k
- R45: value 10 -> 10k
- U8: value NJM4556AD -> TPA6132A2RTER; footprint Package_DIP:DIP-8_W7.62mm -> Package_DFN_QFN:WQFN-16-1EP_3x3mm_P0.5mm_EP1.68x1.68mm
- moved R45 152.7 mm to (217.6, 97.6)
- moved R46 143.2 mm to (216.0, 102.3), turned to 90 degrees
- moved C35 124.7 mm to (98.1, 116.1)
- moved C36 122.1 mm to (101.5, 118.1), turned to 90 degrees
- moved C38 92.8 mm to (95.7, 111.9)
- moved C7 92.3 mm to (105.6, 88.3)
- moved R48 83.8 mm to (170.2, 72.4), turned to 0 degrees
- moved C1 81.5 mm to (138.6, 62.5)
- moved C37 80.9 mm to (104.0, 111.8), turned to 90 degrees
- moved C17 80.6 mm to (112.8, 122.2)
- moved FB1 79.6 mm to (140.0, 58.0)
- moved C2 79.2 mm to (140.4, 56.0)
- moved R47 78.2 mm to (167.4, 89.0)
- moved C9 70.0 mm to (168.0, 53.5), turned to 0 degrees
- moved R32 66.1 mm to (123.8, 106.8)
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Connections:
- C15 pad 1: YM_MOL -> YM_AVCC
- C15 pad 2: FL_IN -> GND
- C16 pad 1: FL_SUM -> YM_AVCC
- C16 pad 2: COLD_L -> GND
- C17 pad 1: HOT_L_R -> YM_MOL
- C17 pad 2: HOT_L_OUT -> FL_IN
- C18 pad 1: COLD_L_R -> FL_SUM
- C18 pad 2: COLD_L_OUT -> COLD_L
- C19 pad 1: COLD_L -> HOT_L_R
- C19 pad 2: VOL_L_IN -> HOT_L_OUT
- C20 pad 1: VOL_L_W -> COLD_L_R
- C20 pad 2: HP_L_IN -> COLD_L_OUT
- C21 pad 1: HP_L_OUT -> COLD_L
- C21 pad 2: HP_L_DC -> VOL_L_IN
- C22 pad 1: YM_MOR -> VOL_L_W
- C22 pad 2: FR_IN -> HP_L_IN
- C23 pad 1: FR_SUM -> YM_MOR
- C23 pad 2: COLD_R -> FR_IN
- C24 pad 1: HOT_R_R -> FR_SUM
- C24 pad 2: HOT_R_OUT -> COLD_R
- C25 pad 1: COLD_R_R -> HOT_R_R
- C25 pad 2: COLD_R_OUT -> HOT_R_OUT
- C26 pad 1: COLD_R -> COLD_R_R
- C26 pad 2: VOL_R_IN -> COLD_R_OUT
- C27 pad 1: VOL_R_W -> COLD_R
- C27 pad 2: HP_R_IN -> VOL_R_IN
- C28 pad 1: HP_R_OUT -> VOL_R_W
- C28 pad 2: HP_R_DC -> HP_R_IN
- C29 pad 2: GNDA -> GND
- C30 pad 2: GNDA -> GND
- C31 pad 1: +4V5A -> HPVDD
- C31 pad 2: GNDA -> GND
- C32 pad 1: +4V5A -> HPVSS
- C32 pad 2: GNDA -> GND
- C33 pad 1: VREF -> HP_CPP
- C33 pad 2: GNDA -> HP_CPN
- C34 pad 1: VREF -> +4V5A
- C34 pad 2: GNDA -> GND
- C35 pad 1: ENC_A -> +4V5A
- C36 pad 1: ENC_B -> +4V5A
- C37 pad 1: +5V -> VREF
- C38 pad 1: +5V -> VREF
- C5 pad 1: +4V5A -> VA_IN
- C5 pad 2: GNDA -> GND
- C6 pad 2: GNDA -> GND
- C7 pad 1: +3V3 -> +4V5A
- C9 pad 1: +5V_YM -> +3V3
- J1 pad 2: SPARE_GP12 -> HP_EN
- J4 pad 3: GNDA -> GND
- J4 pad 6: GNDA -> GND
- J5 pad S: GNDA -> GND
- R21 pad 1: YM_MOL -> +5V_YM
- R21 pad 2: GNDA -> YM_AVCC
- R22 pad 1: FL_IN -> YM_MOL
- R22 pad 2: FL_SUM -> GND
- R23 pad 1: FL_SUM -> FL_IN
- R23 pad 2: COLD_L -> FL_SUM
- R24 pad 1: COLD_L -> FL_SUM
- R24 pad 2: INV_L -> COLD_L
- R25 pad 1: INV_L -> COLD_L
- R25 pad 2: HOT_L -> INV_L
- R26 pad 1: HOT_L -> INV_L
- R26 pad 2: HOT_L_R -> HOT_L
- R27 pad 1: HOT_L_OUT -> HOT_L
- R27 pad 2: GNDA -> HOT_L_R
- R28 pad 1: COLD_L -> HOT_L_OUT
- R28 pad 2: COLD_L_R -> GND
- R29 pad 1: COLD_L_OUT -> COLD_L
- R29 pad 2: GNDA -> COLD_L_R
- R30 pad 1: SLEEVE_L -> COLD_L_OUT
- R30 pad 2: GNDA -> GND
- R31 pad 1: VREF -> SLEEVE_L
- R31 pad 2: HP_L_IN -> GND
- R32 pad 1: HP_L_DC -> YM_MOR
- R32 pad 2: PHONE_L -> GND
- R33 pad 1: HP_L_DC -> FR_IN
- R33 pad 2: GNDA -> FR_SUM
- R34 pad 1: YM_MOR -> FR_SUM
- R34 pad 2: GNDA -> COLD_R
- R35 pad 1: FR_IN -> COLD_R
- R35 pad 2: FR_SUM -> INV_R
- R36 pad 1: FR_SUM -> INV_R
- R36 pad 2: COLD_R -> HOT_R
- R37 pad 1: COLD_R -> HOT_R
- R37 pad 2: INV_R -> HOT_R_R
- R38 pad 1: INV_R -> HOT_R_OUT
- R38 pad 2: HOT_R -> GND
- R39 pad 1: HOT_R -> COLD_R
- R39 pad 2: HOT_R_R -> COLD_R_R
- R40 pad 1: HOT_R_OUT -> COLD_R_OUT
- R40 pad 2: GNDA -> GND
- R41 pad 1: COLD_R -> SLEEVE_R
- R41 pad 2: COLD_R_R -> GND
- R42 pad 1: COLD_R_OUT -> HP_EN
- R42 pad 2: GNDA -> GND
- R43 pad 1: SLEEVE_R -> +4V5A
- R43 pad 2: GNDA -> VREF
- R44 pad 2: HP_R_IN -> GND
- R45 pad 1: HP_R_DC -> +3V3
- R45 pad 2: PHONE_R -> ENC_A
- R46 pad 1: HP_R_DC -> +3V3
- R46 pad 2: GNDA -> ENC_B
- R47 pad 1: +4V5A -> +3V3
- R47 pad 2: VREF -> I2C_SDA
- R48 pad 1: VREF -> +5V
- R48 pad 2: GNDA -> LCD_SDA
- R49 pad 2: ENC_A -> I2C_SCL
- R50 pad 1: +3V3 -> +5V
- R50 pad 2: ENC_B -> LCD_SCL
- U1 pad 2: GNDA -> GND
- U2 pad 16: SPARE_GP12 -> HP_EN
- U5 pad 19: GNDA -> GND
- U5 pad 22: +5V_YM -> YM_AVCC
- U6 pad 4: GNDA -> GND
- U7 pad 4: GNDA -> GND
- U8 pad 1: HP_L_OUT -> HP_L_IN
- U8 pad 2: HP_L_OUT -> GND
- U8 pad 3: HP_L_IN -> GND
- U8 pad 4: GNDA -> HP_R_IN
- U8 pad 5: HP_R_IN -> PHONE_R
- U8 pad 6: HP_R_OUT -> GND
- U8 pad 7: HP_R_OUT -> GND
- U8 pad 8: +4V5A -> HPVSS
Routing:
- net GNDA: track 387.8 -> 0.00 mm
- net GND: track 700.4 -> 917.3 mm, vias 4 -> 334
- net HP_EN: track 0.00 -> 176.9 mm, vias 0 -> 3
- net VA_IN: track 86.3 -> 14.3 mm
- net HOT_R_R: track 41.0 -> 105.9 mm, vias 2 -> 0
- net +5V_YM: track 187.2 -> 130.3 mm, vias 1 -> 3
- net HP_L_IN: track 56.9 -> 11.0 mm, vias 0 -> 2
- net +5V: track 238.5 -> 277.0 mm, vias 6 -> 4
- net +4V5A: track 130.6 -> 93.8 mm, vias 3 -> 4
- net BTN_WRITE: track 198.3 -> 161.6 mm, vias 1 -> 0
- net ENC_B: track 118.6 -> 148.1 mm, vias 2 -> 1
- net HP_R_IN: track 41.5 -> 13.1 mm
- net SPARE_GP12: track 28.2 -> 0.00 mm
- net HP_R_DC: track 28.1 -> 0.00 mm
- net YM_AVCC: track 0.00 -> 26.9 mm
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- removed copper zone on B.Cu, net GNDA
- removed copper zone on F.Cu, net GNDA

Commit message: Rev B layout: wider clearances, no ground traces, 45 degree corners, clean silkscreen
Same circuit and part positions as Rev A, re-routed after the Oct 30 peer review:
- 0.25 mm tracks and gaps, 0.7/0.3 mm vias; 0.2 mm only between U8's own QFN pins
- GND left to the planes; ground vias, stitching and island ties instead of traces
- 90 degree track corners cut into 45 degree bends
- 1.0 mm silkscreen labels clear of pads, parts and edges; outlines trimmed off pads
- DRC (KiCad 7): 0 errors, 0 unconnected, 0 silkscreen warnings; fab files regenerated

Co-Authored-By: Claude Opus 5.5 <noreply@anthropic.com>
Claude-Session: https://claude.ai/code/session_01TDTDVidYRoyJdUGgsyVTSw
Routing:
- net GND: track 917.3 -> 48.8 mm, vias 334 -> 362
- net HOT_R_R: track 105.9 -> 44.3 mm, vias 0 -> 2
- net COLD_L: track 54.7 -> 32.6 mm
- net +5V: track 277.0 -> 256.2 mm, vias 4 -> 3
- net HP_EN: track 176.9 -> 196.2 mm, vias 3 -> 4
- net COLD_R: track 32.8 -> 48.4 mm, vias 4 -> 3
- net MCU_A1: track 51.5 -> 38.0 mm
- net LCD_SCL: track 20.1 -> 33.4 mm, vias 0 -> 1
- net MCU_D3: track 30.6 -> 43.7 mm, vias 0 -> 2
- net MCU_A0: track 41.1 -> 52.2 mm, vias 0 -> 1
- net +5V_YM: track 130.3 -> 141.2 mm, vias 3 -> 4
- net MCU_D1: track 48.5 -> 38.0 mm
- net LCD_SDA: track 18.7 -> 28.9 mm, vias 0 -> 1
- net BTN_WRITE: track 161.6 -> 153.0 mm
- net OSC_OUT: track 23.8 -> 31.2 mm
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Other:
- board text added: "YM2612 Rev B"
- board text removed: "YM2612 Rev A"

Commit message: Silkscreen: add the CTRLVLTS logo above the button row
Co-Authored-By: Claude Opus 5.5 <noreply@anthropic.com>
Claude-Session: https://claude.ai/code/session_01TDTDVidYRoyJdUGgsyVTSw
Other:
- board text added: "[-] CTRLVLTS [+]"
Changed lines of the file:
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@@
   (gr_line (start 59.5 170) (end 50 170)
     (stroke (width 0.1) (type default)) (layer "Edge.Cuts"))
+  (gr_text "[-] CTRLVLTS [+]" (at 157 128) (layer "F.SilkS")
+    (effects (font (size 2.2 2.2) (thickness 0.33)))
+  )
   (gr_text "BAL L     BAL R" (at 62 76.5) (layer "F.SilkS")
     (effects (font (size 1.2 1.2) (thickness 0.18)) (justify left))
